Commit message: fixed collision typo for gazebo

File: my_rb1_description/urdf/my_rb1_robot.urdf (robot description, URDF)
Before this commit: robot my_rb1_robot, 7 links, 6 joints
Links:
- link link_base: geometry collision cylinder length=.3 radius=.25; visual cylinder length=.3 radius=.25
- link link_base_footprint: mass .1 -> 0; geometry 
- link link_caster_back: mass 1 -> .1; geometry collision sphere radius=.05; visual sphere radius=.05
- link link_caster_front: mass 1 -> .1; geometry collision sphere radius=.05; visual sphere radius=.05
- link link_left_wheel: mass 1 -> .1; geometry collision cylinder length=.05 radius=.05; visual cylinder length=.05 radius=.05
- link link_right_wheel: mass 1 -> .1; geometry collision cylinder length=.05 radius=.05; visual cylinder length=.05 radius=.05

Commit message: added ros plugins

File: my_rb1_description/urdf/my_rb1_robot.urdf (robot description, URDF)
Before this commit: robot my_rb1_robot, 7 links, 6 joints
Joints:
- joint laser_scan_chassis_joint: origin xyz=.25 0 .075 rpy=0 1.57 0 -> xyz=.25 0 .075 rpy=0 0 0
- joint left_wheel_joint: origin xyz=0.0 -0.2 -0.15 rpy=0 0 3.14 -> xyz=0.0 -0.2 -0.15 rpy=0 0 0
